Commit message: update xela_models

File: urdf/4x4.urdf (robot description, URDF)
Before this commit: robot 4x4, 51 links, 50 joints
Links:
- link 1_4x4_base_link: geometry collision mesh filename=file://$(find xela_models)/mesh/4x4.stl scale=1 1 1; visual mesh filename=file://$(find xela_models)/mesh/4x4.stl scale=1 1 1

File: urdf/allegro_hand_right.xacro (robot description, xacro)
@@ -9,7 +9,8 @@
 Palm sensors can be disabled by setting palm to 0
 -->
-	<xacro:allegro_hand_right sequence="" tips="curved" parent="world" defaultnames="1" baseispalm="1" />
+	<!-- <xacro:allegro_hand_right sequence="" tips="curved" parent="world" defaultnames="1" baseispalm="1" /> -->
   <!-- Enable the following 2 if you would like to see different options the same time -->
 	<!-- <xacro:allegro_hand_right sequence="2" parent="world" x="0.2" tips="curved" /> -->
 	<!-- <xacro:allegro_hand_right sequence="3" parent="world" x="-0.2" covers="0" palm="0" phalanges="0" tips="default"/> -->
+	<xacro:allegro_hand_right sequence="" tips="curved" parent="world" defaultnames="1"/>
 </robot>

File: urdf/xela.xacro (robot description, xacro)
@@ -108,5 +108,5 @@
         <origin xyz="0 0 0" rpy="0 0 0" />
         <geometry>
-          <mesh filename="package://xela_models/mesh/ft_f.stl"/>
+          <mesh filename="file://$(find xela_models)/mesh/ft_f.stl"/>
         </geometry>
       </collision>
@@ -114,5 +114,5 @@
         <origin xyz="0 0 0" rpy="0 0 0" />
         <geometry>
-          <mesh filename="package://xela_models/mesh/ft_f.stl"/>
+          <mesh filename="file://$(find xela_models)/mesh/ft_f.stl"/>
         </geometry>
         <material name="${col}"/>
@@ -182,5 +182,5 @@
         <origin xyz="0 0 0" rpy="0 0 0" />
         <geometry>
-          <mesh filename="package://xela_models/mesh/ft_c.stl"/>
+          <mesh filename="file://$(find xela_models)/mesh/ft_c.stl"/>
         </geometry>
       </collision>
@@ -188,5 +188,5 @@
         <origin xyz="0 0 0" rpy="0 0 0" />
         <geometry>
-          <mesh filename="package://xela_models/mesh/ft_c.stl"/>
+          <mesh filename="file://$(find xela_models)/mesh/ft_c.stl"/>
         </geometry>
         <material name="${col}"/>
@@ -243,5 +243,5 @@
         <origin xyz="0 0 0" rpy="0 0 0" />
         <geometry>
-          <mesh filename="package://xela_models/mesh/allegro/ahft_default.STL"/>
+          <mesh filename="file://$(find xela_models)/mesh/allegro/ahft_default.STL"/>
         </geometry>
       </collision>
@@ -249,5 +249,5 @@
         <origin xyz="0 0 0" rpy="0 0 0" />
         <geometry>
-          <mesh filename="package://xela_models/mesh/allegro/ahft_default.STL"/>
+          <mesh filename="file://$(find xela_models)/mesh/allegro/ahft_default.STL"/>
         </geometry>
         <material name="${col}"/>
@@ -272,5 +272,5 @@
         <origin xyz="0 0 0" rpy="0 0 0" />
         <geometry>
-          <mesh filename="package://xela_models/mesh/4x4.stl"/>
+          <mesh filename="file://$(find xela_models)/mesh/4x4.stl"/>
         </geometry>
       </collision>
@@ -279,5 +279,5 @@
           <origin xyz="0 0 0" rpy="0 0 0" />
           <geometry>
-            <mesh filename="package://xela_models/mesh/4x4.stl"/>
+            <mesh filename="file://$(find xela_models)/mesh/4x4.stl"/>
           </geometry>
           <material name="${col}"/>
@@ -321,5 +321,5 @@
         <origin xyz="0 0 0" rpy="0 0 0" />
         <geometry>
-          <mesh filename="package://xela_models/mesh/1x6.stl"/>
+          <mesh filename="file://$(find xela_models)/mesh/1x6.stl"/>
         </geometry>
       </collision>
@@ -328,5 +328,5 @@
           <origin xyz="0 0 0" rpy="0 0 0" />
           <geometry>
-            <mesh filename="package://xela_models/mesh/1x6.stl"/>
+            <mesh filename="file://$(find xela_models)/mesh/1x6.stl"/>
           </geometry>
           <material name="${col}"/>
@@ -360,5 +360,5 @@
         <origin xyz="0 0 0" rpy="0 0 0" />
         <geometry>
-          <mesh filename="package://xela_models/mesh/4x6.stl"/>
+          <mesh filename="file://$(find xela_models)/mesh/4x6.stl"/>
         </geometry>
       </collision>
@@ -367,5 +367,5 @@
           <origin xyz="0 0 0" rpy="0 0 0" />
           <geometry>
-            <mesh filename="package://xela_models/mesh/4x6.stl"/>
+            <mesh filename="file://$(find xela_models)/mesh/4x6.stl"/>
           </geometry>
           <material name="${col}"/>
@@ -419,8 +419,8 @@
         <geometry>
           <xacro:if value="${palm == 1}">
-            <mesh filename="package://xela_models/mesh/allegro/base.stl" />
+            <mesh filename="file://$(find xela_models)/mesh/allegro/base.stl" />
           </xacro:if>
           <xacro:if value="${palm != 1}">
-            <mesh filename="package://xela_models/mesh/allegro/base_ns.stl"/>
+            <mesh filename="file://$(find xela_models)/mesh/allegro/base_ns.stl"/>
           </xacro:if>
         </geometry>
@@ -579,5 +579,5 @@
         <visual>
           <geometry>
-            <mesh filename="package://xela_models/mesh/allegro/link_0.0_ext.STL" />
+            <mesh filename="file://$(find xela_models)/mesh/allegro/link_0.0_ext.STL" />
           </geometry>
           <material name="grey"/>
@@ -606,8 +606,8 @@
           <geometry>
             <xacro:if value="${phalanges == 1}">
-              <mesh filename="package://xela_models/mesh/allegro/link_1.1.stl" />
+              <mesh filename="file://$(find xela_models)/mesh/allegro/link_1.1.stl" />
             </xacro:if>
             <xacro:if value="${phalanges != 1}">
-              <mesh filename="package://xela_models/mesh/allegro/link_1_ns.stl"/>
+              <mesh filename="file://$(find xela_models)/mesh/allegro/link_1_ns.stl"/>
             </xacro:if>
           </geometry>
@@ -648,5 +648,5 @@
           <visual>
             <geometry>
-              <mesh filename="package://xela_models/mesh/allegro/link_1_cover.stl" />
+              <mesh filename="file://$(find xela_models)/mesh/allegro/link_1_cover.stl" />
             </geometry>
             <material name="red"/>
@@ -654,5 +654,5 @@
           <collision>
             <geometry>
-              <mesh filename="package://xela_models/mesh/allegro/link_1_cover.stl" />
+              <mesh filename="file://$(find xela_models)/mesh/allegro/link_1_cover.stl" />
             </geometry>
             <origin rpy="0 0 0" xyz="0 0 ${0.0177/2}"/>
@@ -681,8 +681,8 @@
           <geometry>
             <xacro:if value="${phalanges == 1}">
-              <mesh filename="package://xela_models/mesh/allegro/link_2.1.stl" />
+              <mesh filename="file://$(find xela_models)/mesh/allegro/link_2.1.stl" />
             </xacro:if>
             <xacro:if value="${phalanges != 1}">
-              <mesh filename="package://xela_models/mesh/allegro/link_2_ns.stl"/>
+              <mesh filename="file://$(find xela_models)/mesh/allegro/link_2_ns.stl"/>
             </xacro:if>
           </geometry>
@@ -723,5 +723,5 @@
           <visual>
             <geometry>
-              <mesh filename="package://xela_models/mesh/allegro/link_2_cover.stl" />
+              <mesh filename="file://$(find xela_models)/mesh/allegro/link_2_cover.stl" />
             </geometry>
             <material name="red"/>
@@ -729,5 +729,5 @@
           <collision>
             <geometry>
-              <mesh filename="package://xela_models/mesh/allegro/link_2_cover.stl" />
+              <mesh filename="file://$(find xela_models)/mesh/allegro/link_2_cover.stl" />
             </geometry>
             <origin rpy="0 0 0" xyz="0 0 ${0.0514/2}"/>
@@ -753,5 +753,5 @@
         <visual>
           <geometry>
-            <mesh filename="package://xela_models/mesh/allegro/link_3.0.STL" />
+            <mesh filename="file://$(find xela_models)/mesh/allegro/link_3.0.STL" />
           </geometry>
           <material name="black" />
@@ -807,5 +807,5 @@
         <visual>
           <geometry>
-            <mesh filename="package://xela_models/mesh/allegro/link_12.0_right.STL" />
+            <mesh filename="file://$(find xela_models)/mesh/allegro/link_12.0_right.STL" />
           </geometry>
           <material name="grey" />
@@ -833,5 +833,5 @@
         <visual>
           <geometry>
-            <mesh filename="package://xela_models/mesh/allegro/link_13.0.STL" />
+            <mesh filename="file://$(find xela_models)/mesh/allegro/link_13.0.STL" />
           </geometry>
           <material name="grey" />
@@ -853,5 +853,5 @@
           <visual>
             <geometry>
-              <mesh filename="package://xela_models/mesh/allegro/thumb_1_cover.stl" />
+              <mesh filename="file://$(find xela_models)/mesh/allegro/thumb_1_cover.stl" />
             </geometry>
             <material name="red"/>
@@ -859,5 +859,5 @@
           <collision>
             <geometry>
-              <mesh filename="package://xela_models/mesh/allegro/thumb_1_cover.stl" />
+              <mesh filename="file://$(find xela_models)/mesh/allegro/thumb_1_cover.stl" />
             </geometry>
             <origin rpy="0 0 0" xyz="0 0 0"/>
@@ -881,8 +881,8 @@
           <geometry>
             <xacro:if value="${phalanges == 1}">
-              <mesh filename="package://xela_models/mesh/allegro/thumb_1.1.stl"/>
+              <mesh filename="file://$(find xela_models)/mesh/allegro/thumb_1.1.stl"/>
             </xacro:if>
             <xacro:if value="${phalanges != 1}">
-              <mesh filename="package://xela_models/mesh/allegro/thumb_1.1_ns.stl"/>
+              <mesh filename="file://$(find xela_models)/mesh/allegro/thumb_1.1_ns.stl"/>
             </xacro:if>
           </geometry>
@@ -923,5 +923,5 @@
           <visual>
             <geometry>
-              <mesh filename="package://xela_models/mesh/allegro/thumb_2_cover.stl" />
+              <mesh filename="file://$(find xela_models)/mesh/allegro/thumb_2_cover.stl" />
             </geometry>
             <material name="red"/>
@@ -929,5 +929,5 @@
           <collision>
             <geometry>
-              <mesh filename="package://xela_models/mesh/allegro/thumb_2_cover.stl" />
+              <mesh filename="file://$(find xela_models)/mesh/allegro/thumb_2_cover.stl" />
             </geometry>
             <origin rpy="0 0 0" xyz="0 0 0"/>
@@ -954,8 +954,8 @@
           <geometry>
             <xacro:if value="${phalanges == 1}">
-              <mesh filename="package://xela_models/mesh/allegro/thumb_2.1.stl"/>
+              <mesh filename="file://$(find xela_models)/mesh/allegro/thumb_2.1.stl"/>
             </xacro:if>
             <xacro:if value="${phalanges != 1}">
-              <mesh filename="package://xela_models/mesh/allegro/thumb_1.2_ns.stl"/>
+              <mesh filename="file://$(find xela_models)/mesh/allegro/thumb_1.2_ns.stl"/>
             </xacro:if>
           </geometry>
