Commit message: rename link names

File: urdf/my_xela_allegro.urdf (robot description, URDF)
Before this commit: robot allegro_hand_right, 44 links, 43 joints
Links:
- removed link 0aftc_palm_link
- removed link 1aftc_palm_link
- removed link 2aftc_palm_link
- removed link 3aftc_palm_link
- removed link ahr_palm_1_4x6_palm_link
- removed link ahr_palm_2_4x6_palm_link
- removed link ahr_palm_3_4x6_palm_link
- removed link link_0
- removed link link_1
- removed link link_10
- removed link link_10_4x4_palm_link
- removed link link_10_cover
- removed link link_11
- removed link link_12
- removed link link_13
- removed link link_14
- removed link link_14_4x4_palm_link
- removed link link_14_cover
- removed link link_15
- removed link link_15_4x4_palm_link
- removed link link_15_cover
- removed link link_1A_4x4_palm_link
- removed link link_1B_4x4_palm_link
- removed link link_1_cover
- removed link link_2
- removed link link_2_4x4_palm_link
- removed link link_2_cover
- removed link link_3
- removed link link_4
- removed link link_5
- removed link link_5A_4x4_palm_link
- removed link link_5B_4x4_palm_link
- removed link link_5_cover
- removed link link_6
- removed link link_6_4x4_palm_link
- removed link link_6_cover
- removed link link_7
- removed link link_8
- removed link link_9
- removed link link_9A_4x4_palm_link
- removed link link_9B_4x4_palm_link
- removed link link_9_cover
- added link cover_index_1; collision mesh filename=package://xela_models/mesh/allegro/link_1_cover.stl; visual mesh filename=package://xela_models/mesh/allegro/link_1_cover.stl
- added link cover_index_2; collision mesh filename=package://xela_models/mesh/allegro/link_2_cover.stl; visual mesh filename=package://xela_models/mesh/allegro/link_2_cover.stl
- added link cover_middle_1; collision mesh filename=package://xela_models/mesh/allegro/link_1_cover.stl; visual mesh filename=package://xela_models/mesh/allegro/link_1_cover.stl
- added link cover_middle_2; collision mesh filename=package://xela_models/mesh/allegro/link_2_cover.stl; visual mesh filename=package://xela_models/mesh/allegro/link_2_cover.stl
- added link cover_ring_1; collision mesh filename=package://xela_models/mesh/allegro/link_1_cover.stl; visual mesh filename=package://xela_models/mesh/allegro/link_1_cover.stl
- added link cover_ring_2; collision mesh filename=package://xela_models/mesh/allegro/link_2_cover.stl; visual mesh filename=package://xela_models/mesh/allegro/link_2_cover.stl
- added link cover_thumb_1; collision mesh filename=package://xela_models/mesh/allegro/thumb_1_cover.stl; visual mesh filename=package://xela_models/mesh/allegro/thumb_1_cover.stl
- added link cover_thumb_2; collision mesh filename=package://xela_models/mesh/allegro/thumb_2_cover.stl; visual mesh filename=package://xela_models/mesh/allegro/thumb_2_cover.stl
- added link index_fingertip_link; collision mesh filename=package://xela_models/mesh/ft_c.stl; visual mesh filename=package://xela_models/mesh/ft_c.stl
- added link index_link_1, mass 0.0127; collision box size=0.0196 0.0275 0.0164; visual mesh filename=package://xela_models/mesh/allegro/link_0.0_ext.STL
- added link index_link_2, mass 0.0809; collision box size=0.0196 0.0275 0.0164; visual mesh filename=package://xela_models/mesh/allegro/link_1.0.stl
- added link index_link_3, mass 0.0447; collision box size=0.0196 0.0275 0.054; visual mesh filename=package://xela_models/mesh/allegro/link_2.0.stl
- added link index_link_4, mass 0.0404; collision box size=0.0196 0.0275 0.026399999999999996; visual mesh filename=package://xela_models/mesh/allegro/link_3.0.STL
- added link middle_fingertip_link; collision mesh filename=package://xela_models/mesh/ft_c.stl; visual mesh filename=package://xela_models/mesh/ft_c.stl
- added link middle_link_1, mass 0.0127; collision box size=0.0196 0.0275 0.0164; visual mesh filename=package://xela_models/mesh/allegro/link_0.0_ext.STL
- added link middle_link_2, mass 0.0809; collision box size=0.0196 0.0275 0.0164; visual mesh filename=package://xela_models/mesh/allegro/link_1.0.stl
- added link middle_link_3, mass 0.0447; collision box size=0.0196 0.0275 0.054; visual mesh filename=package://xela_models/mesh/allegro/link_2.0.stl
- added link middle_link_4, mass 0.0404; collision box size=0.0196 0.0275 0.026399999999999996; visual mesh filename=package://xela_models/mesh/allegro/link_3.0.STL
- added link ring_fingertip_link; collision mesh filename=package://xela_models/mesh/ft_c.stl; visual mesh filename=package://xela_models/mesh/ft_c.stl
- added link ring_link_1, mass 0.0127; collision box size=0.0196 0.0275 0.0164; visual mesh filename=package://xela_models/mesh/allegro/link_0.0_ext.STL
- added link ring_link_2, mass 0.0809; collision box size=0.0196 0.0275 0.0164; visual mesh filename=package://xela_models/mesh/allegro/link_1.0.stl
- added link ring_link_3, mass 0.0447; collision box size=0.0196 0.0275 0.054; visual mesh filename=package://xela_models/mesh/allegro/link_2.0.stl
- added link ring_link_4, mass 0.0404; collision box size=0.0196 0.0275 0.026399999999999996; visual mesh filename=package://xela_models/mesh/allegro/link_3.0.STL
- added link sensor_index_1; collision mesh filename=package://xela_models/mesh/4x4.stl; visual mesh filename=package://xela_models/mesh/4x4.stl
- added link sensor_index_2; collision mesh filename=package://xela_models/mesh/4x4.stl; visual mesh filename=package://xela_models/mesh/4x4.stl
- added link sensor_index_3; collision mesh filename=package://xela_models/mesh/4x4.stl; visual mesh filename=package://xela_models/mesh/4x4.stl
- added link sensor_middle_1; collision mesh filename=package://xela_models/mesh/4x4.stl; visual mesh filename=package://xela_models/mesh/4x4.stl
- added link sensor_middle_2; collision mesh filename=package://xela_models/mesh/4x4.stl; visual mesh filename=package://xela_models/mesh/4x4.stl
- added link sensor_middle_3; collision mesh filename=package://xela_models/mesh/4x4.stl; visual mesh filename=package://xela_models/mesh/4x4.stl
- added link sensor_palm_bottom_left; collision mesh filename=package://xela_models/mesh/4x6.stl; visual mesh filename=package://xela_models/mesh/4x6.stl
- added link sensor_palm_top_left; collision mesh filename=package://xela_models/mesh/4x6.stl; visual mesh filename=package://xela_models/mesh/4x6.stl
- added link sensor_palm_top_right; collision mesh filename=package://xela_models/mesh/4x6.stl; visual mesh filename=package://xela_models/mesh/4x6.stl
- added link sensor_ring_1; collision mesh filename=package://xela_models/mesh/4x4.stl; visual mesh filename=package://xela_models/mesh/4x4.stl
- added link sensor_ring_2; collision mesh filename=package://xela_models/mesh/4x4.stl; visual mesh filename=package://xela_models/mesh/4x4.stl
- added link sensor_ring_3; collision mesh filename=package://xela_models/mesh/4x4.stl; visual mesh filename=package://xela_models/mesh/4x4.stl
- added link sensor_thumb_1; collision mesh filename=package://xela_models/mesh/4x4.stl; visual mesh filename=package://xela_models/mesh/4x4.stl
- added link sensor_thumb_2; collision mesh filename=package://xela_models/mesh/4x4.stl; visual mesh filename=package://xela_models/mesh/4x4.stl
- added link thumb_fingertip_link; collision mesh filename=package://xela_models/mesh/ft_c.stl; visual mesh filename=package://xela_models/mesh/ft_c.stl
- added link thumb_link_1, mass 0.0176; collision box size=0.0358 0.034 0.0455; visual mesh filename=package://xela_models/mesh/allegro/link_12.0_right.STL
- added link thumb_link_2, mass 0.0127; collision box size=0.0196 0.0275 0.0177; visual mesh filename=package://xela_models/mesh/allegro/link_0.0_ext.STL
- added link thumb_link_3, mass 0.0457; collision box size=0.0196 0.0275 0.0514; visual mesh filename=package://xela_models/mesh/allegro/thumb_1.0.stl
- added link thumb_link_4, mass 0.0753; collision box size=0.0196 0.0275 0.042300000000000004; visual mesh filename=package://xela_models/mesh/allegro/thumb_2.0.stl
Joints:
- removed joint 0aftc_fixed
- removed joint 1aftc_fixed
- removed joint 2aftc_fixed
- removed joint 3aftc_fixed
- added joint index_fingertip_fixed_joint: type fixed, parent index_link_4, child index_fingertip_link, origin xyz=-0.013 0.0 0.016 rpy=1.5707963267948966 0.0 1.5707963267948966
- added joint middle_fingertip_fixed_joint: type fixed, parent middle_link_4, child middle_fingertip_link, origin xyz=-0.013 0.0 0.016 rpy=1.5707963267948966 0.0 1.5707963267948966
- added joint ring_fingertip_fixed_joint: type fixed, parent ring_link_4, child ring_fingertip_link, origin xyz=-0.013 0.0 0.016 rpy=1.5707963267948966 0.0 1.5707963267948966
- added joint thumb_fingertip_fixed_joint: type fixed, parent thumb_link_4, child thumb_fingertip_link, origin xyz=-0.013 0.0 0.0315 rpy=1.5707963267948966 0.0 1.5707963267948966
- joint ahr_palm_1_4x6_fixed: child ahr_palm_1_4x6_palm_link -> sensor_palm_top_left
- joint ahr_palm_2_4x6_fixed: child ahr_palm_2_4x6_palm_link -> sensor_palm_top_right
- joint ahr_palm_3_4x6_fixed: child ahr_palm_3_4x6_palm_link -> sensor_palm_bottom_left
- joint joint_0: child link_0 -> index_link_1
- joint joint_1: child link_1 -> index_link_2; parent link_0 -> index_link_1
- joint joint_10: child link_10 -> ring_link_3; parent link_9 -> ring_link_2
- joint joint_11: child link_11 -> ring_link_4; parent link_10 -> ring_link_3
- joint joint_12: child link_12 -> thumb_link_1
- joint joint_13: child link_13 -> thumb_link_2; parent link_12 -> thumb_link_1
- joint joint_14: child link_14 -> thumb_link_3; parent link_13 -> thumb_link_2
- joint joint_15: child link_15 -> thumb_link_4; parent link_14 -> thumb_link_3
- joint joint_2: child link_2 -> index_link_3; parent link_1 -> index_link_2
- joint joint_3: child link_3 -> index_link_4; parent link_2 -> index_link_3
- joint joint_4: child link_4 -> middle_link_1
- joint joint_5: child link_5 -> middle_link_2; parent link_4 -> middle_link_1
- joint joint_6: child link_6 -> middle_link_3; parent link_5 -> middle_link_2
- joint joint_7: child link_7 -> middle_link_4; parent link_6 -> middle_link_3
- joint joint_8: child link_8 -> ring_link_1
- joint joint_9: child link_9 -> ring_link_2; parent link_8 -> ring_link_1
- joint link_10_4x4_fixed: child link_10_4x4_palm_link -> sensor_ring_3; parent link_10 -> ring_link_3
- joint link_10_cover_joint: child link_10_cover -> cover_ring_2; parent link_10 -> ring_link_3
- joint link_14_4x4_fixed: child link_14_4x4_palm_link -> sensor_thumb_1; parent link_14 -> thumb_link_3
- joint link_14_cover_joint: child link_14_cover -> cover_thumb_1; parent link_14 -> thumb_link_3
- joint link_15_4x4_fixed: child link_15_4x4_palm_link -> sensor_thumb_2; parent link_15 -> thumb_link_4
- joint link_15_cover_joint: child link_15_cover -> cover_thumb_2; parent link_15 -> thumb_link_4
- joint link_1A_4x4_fixed: child link_1A_4x4_palm_link -> sensor_index_2; parent link_1 -> index_link_2
- joint link_1B_4x4_fixed: child link_1B_4x4_palm_link -> sensor_index_1; parent link_1 -> index_link_2
- joint link_1_cover_joint: child link_1_cover -> cover_index_1; parent link_1 -> index_link_2
- joint link_2_4x4_fixed: child link_2_4x4_palm_link -> sensor_index_3; parent link_2 -> index_link_3
- joint link_2_cover_joint: child link_2_cover -> cover_index_2; parent link_2 -> index_link_3
- joint link_5A_4x4_fixed: child link_5A_4x4_palm_link -> sensor_middle_2; parent link_5 -> middle_link_2
- joint link_5B_4x4_fixed: child link_5B_4x4_palm_link -> sensor_middle_1; parent link_5 -> middle_link_2
- joint link_5_cover_joint: child link_5_cover -> cover_middle_1; parent link_5 -> middle_link_2
- joint link_6_4x4_fixed: child link_6_4x4_palm_link -> sensor_middle_3; parent link_6 -> middle_link_3
- joint link_6_cover_joint: child link_6_cover -> cover_middle_2; parent link_6 -> middle_link_3
- joint link_9A_4x4_fixed: child link_9A_4x4_palm_link -> sensor_ring_2; parent link_9 -> ring_link_2
- joint link_9B_4x4_fixed: child link_9B_4x4_palm_link -> sensor_ring_1; parent link_9 -> ring_link_2
- joint link_9_cover_joint: child link_9_cover -> cover_ring_1; parent link_9 -> ring_link_2

Commit message: rename to isaaclab compatible urdf

File: urdf/my_xela_allegro.urdf (robot description, URDF)
Before this commit: robot allegro_hand_right, 44 links, 43 joints
Links:
- link index_link_1: geometry collision box size=0.0196 0.0275 0.0164; visual mesh filename=package://xela_models/mesh/allegro/link_0_ext.STL
- link index_link_2: geometry collision box size=0.0196 0.0275 0.0164; visual mesh filename=package://xela_models/mesh/allegro/link_1.stl
- link index_link_3: geometry collision box size=0.0196 0.0275 0.054; visual mesh filename=package://xela_models/mesh/allegro/link_2.stl
- link index_link_4: geometry collision box size=0.0196 0.0275 0.026399999999999996; visual mesh filename=package://xela_models/mesh/allegro/link_3.STL
- link middle_link_1: geometry collision box size=0.0196 0.0275 0.0164; visual mesh filename=package://xela_models/mesh/allegro/link_0_ext.STL
- link middle_link_2: geometry collision box size=0.0196 0.0275 0.0164; visual mesh filename=package://xela_models/mesh/allegro/link_1.stl
- link middle_link_3: geometry collision box size=0.0196 0.0275 0.054; visual mesh filename=package://xela_models/mesh/allegro/link_2.stl
- link middle_link_4: geometry collision box size=0.0196 0.0275 0.026399999999999996; visual mesh filename=package://xela_models/mesh/allegro/link_3.STL
- link ring_link_1: geometry collision box size=0.0196 0.0275 0.0164; visual mesh filename=package://xela_models/mesh/allegro/link_0_ext.STL
- link ring_link_2: geometry collision box size=0.0196 0.0275 0.0164; visual mesh filename=package://xela_models/mesh/allegro/link_1.stl
- link ring_link_3: geometry collision box size=0.0196 0.0275 0.054; visual mesh filename=package://xela_models/mesh/allegro/link_2.stl
- link ring_link_4: geometry collision box size=0.0196 0.0275 0.026399999999999996; visual mesh filename=package://xela_models/mesh/allegro/link_3.STL
- link sensor_index_1: geometry collision mesh filename=package://xela_models/mesh/sensor_4x4.stl; visual mesh filename=package://xela_models/mesh/sensor_4x4.stl
- link sensor_index_2: geometry collision mesh filename=package://xela_models/mesh/sensor_4x4.stl; visual mesh filename=package://xela_models/mesh/sensor_4x4.stl
- link sensor_index_3: geometry collision mesh filename=package://xela_models/mesh/sensor_4x4.stl; visual mesh filename=package://xela_models/mesh/sensor_4x4.stl
- link sensor_middle_1: geometry collision mesh filename=package://xela_models/mesh/sensor_4x4.stl; visual mesh filename=package://xela_models/mesh/sensor_4x4.stl
- link sensor_middle_2: geometry collision mesh filename=package://xela_models/mesh/sensor_4x4.stl; visual mesh filename=package://xela_models/mesh/sensor_4x4.stl
- link sensor_middle_3: geometry collision mesh filename=package://xela_models/mesh/sensor_4x4.stl; visual mesh filename=package://xela_models/mesh/sensor_4x4.stl
- link sensor_palm_bottom_left: geometry collision mesh filename=package://xela_models/mesh/sensor_4x6.stl; visual mesh filename=package://xela_models/mesh/sensor_4x6.stl
- link sensor_palm_top_left: geometry collision mesh filename=package://xela_models/mesh/sensor_4x6.stl; visual mesh filename=package://xela_models/mesh/sensor_4x6.stl
- link sensor_palm_top_right: geometry collision mesh filename=package://xela_models/mesh/sensor_4x6.stl; visual mesh filename=package://xela_models/mesh/sensor_4x6.stl
- link sensor_ring_1: geometry collision mesh filename=package://xela_models/mesh/sensor_4x4.stl; visual mesh filename=package://xela_models/mesh/sensor_4x4.stl
- link sensor_ring_2: geometry collision mesh filename=package://xela_models/mesh/sensor_4x4.stl; visual mesh filename=package://xela_models/mesh/sensor_4x4.stl
- link sensor_ring_3: geometry collision mesh filename=package://xela_models/mesh/sensor_4x4.stl; visual mesh filename=package://xela_models/mesh/sensor_4x4.stl
- link sensor_thumb_1: geometry collision mesh filename=package://xela_models/mesh/sensor_4x4.stl; visual mesh filename=package://xela_models/mesh/sensor_4x4.stl
- link sensor_thumb_2: geometry collision mesh filename=package://xela_models/mesh/sensor_4x4.stl; visual mesh filename=package://xela_models/mesh/sensor_4x4.stl
- link thumb_link_1: geometry collision box size=0.0358 0.034 0.0455; visual mesh filename=package://xela_models/mesh/allegro/link_12_right.STL
- link thumb_link_2: geometry collision box size=0.0196 0.0275 0.0177; visual mesh filename=package://xela_models/mesh/allegro/link_0_ext.STL
- link thumb_link_3: geometry collision box size=0.0196 0.0275 0.0514; visual mesh filename=package://xela_models/mesh/allegro/thumb_1.stl
- link thumb_link_4: geometry collision box size=0.0196 0.0275 0.042300000000000004; visual mesh filename=package://xela_models/mesh/allegro/thumb_2.stl
