Commit message: add palm sensors

File: urdf/tactile_xela_allegro.urdf (robot description, URDF)
Before this commit: robot xela_allegro_hand, 21 links, 20 joints
Links:
- added link palm_sensor_1_link, mass 0; collision box size=0.001 0.0405 0.026; visual box size=0.001 0.0405 0.026
- added link palm_sensor_2_link, mass 0; collision box size=0.001 0.0405 0.026; visual box size=0.001 0.0405 0.026
- added link palm_sensor_3_link, mass 0; collision box size=0.001 0.0405 0.026; visual box size=0.001 0.0405 0.026
Joints:
- added joint palm_sensor_1_joint: type fixed, parent allegro_base_link, child palm_sensor_1_link, origin xyz=0 0 0 rpy=0 0 0
- added joint palm_sensor_2_joint: type fixed, parent allegro_base_link, child palm_sensor_2_link, origin xyz=0 0 0 rpy=0 0 0
- added joint palm_sensor_3_joint: type fixed, parent allegro_base_link, child palm_sensor_3_link, origin xyz=0 0 0 rpy=0 0 0

Commit message: add all other sensors

File: urdf/tactile_xela_allegro.urdf (robot description, URDF)
Before this commit: robot xela_allegro_hand, 24 links, 23 joints
Links:
- added link index_sensor_2_link, mass 0; collision box size=0.001 0.018 0.0205; visual box size=0.001 0.018 0.0205
- added link index_sensor_3_link, mass 0; collision box size=0.001 0.018 0.0205; visual box size=0.001 0.018 0.0205
- added link index_sensor_4_link, mass 0; collision box size=0.001 0.018 0.0205; visual box size=0.001 0.018 0.0205
- added link middle_sensor_2_link, mass 0; collision box size=0.001 0.018 0.0205; visual box size=0.001 0.018 0.0205
- added link middle_sensor_3_link, mass 0; collision box size=0.001 0.018 0.0205; visual box size=0.001 0.018 0.0205
- added link middle_sensor_4_link, mass 0; collision box size=0.001 0.018 0.0205; visual box size=0.001 0.018 0.0205
- added link ring_sensor_2_link, mass 0; collision box size=0.001 0.018 0.0205; visual box size=0.001 0.018 0.0205
- added link ring_sensor_3_link, mass 0; collision box size=0.001 0.018 0.0205; visual box size=0.001 0.018 0.0205
- added link ring_sensor_4_link, mass 0; collision box size=0.001 0.018 0.0205; visual box size=0.001 0.018 0.0205
- added link thumb_sensor_2_link, mass 0; collision box size=0.001 0.018 0.0205; visual box size=0.001 0.018 0.0205
- added link thumb_sensor_3_link, mass 0; collision box size=0.001 0.018 0.0205; visual box size=0.001 0.018 0.0205
Joints:
- added joint index_sensor_2_joint: type fixed, parent allegro_link_13, child index_sensor_2_link, origin xyz=0 0 0 rpy=0 0 0
- added joint index_sensor_3_joint: type fixed, parent allegro_link_12, child index_sensor_3_link, origin xyz=0 0 0 rpy=0 0 0
- added joint index_sensor_4_joint: type fixed, parent allegro_link_12, child index_sensor_4_link, origin xyz=0 0 0 rpy=0 0 0
- added joint middle_sensor_2_joint: type fixed, parent allegro_link_23, child middle_sensor_2_link, origin xyz=0 0 0 rpy=0 0 0
- added joint middle_sensor_3_joint: type fixed, parent allegro_link_22, child middle_sensor_3_link, origin xyz=0 0 0 rpy=0 0 0
- added joint middle_sensor_4_joint: type fixed, parent allegro_link_22, child middle_sensor_4_link, origin xyz=0 0 0 rpy=0 0 0
- added joint ring_sensor_2_joint: type fixed, parent allegro_link_33, child ring_sensor_2_link, origin xyz=0 0 0 rpy=0 0 0
- added joint ring_sensor_3_joint: type fixed, parent allegro_link_32, child ring_sensor_3_link, origin xyz=0 0 0 rpy=0 0 0
- added joint ring_sensor_4_joint: type fixed, parent allegro_link_32, child ring_sensor_4_link, origin xyz=0 0 0 rpy=0 0 0
- added joint thumb_sensor_2_joint: type fixed, parent allegro_link_44, child thumb_sensor_2_link, origin xyz=0 0 0 rpy=0 0 0
- added joint thumb_sensor_3_joint: type fixed, parent allegro_link_43, child thumb_sensor_3_link, origin xyz=0 0 0 rpy=0 0 0

Commit message: add mass and inertia to sensor bodies

File: urdf/tactile_xela_allegro.urdf (robot description, URDF)
Before this commit: robot xela_allegro_hand, 35 links, 34 joints
Links:
- link index_sensor_2_link: mass 0 -> 0.01
- link index_sensor_3_link: mass 0 -> 0.01
- link index_sensor_4_link: mass 0 -> 0.01
- link middle_sensor_2_link: mass 0 -> 0.01
- link middle_sensor_3_link: mass 0 -> 0.01
- link middle_sensor_4_link: mass 0 -> 0.01
- link palm_sensor_1_link: mass 0 -> 0.01
- link palm_sensor_2_link: mass 0 -> 0.01
- link palm_sensor_3_link: mass 0 -> 0.01
- link ring_sensor_2_link: mass 0 -> 0.01
- link ring_sensor_3_link: mass 0 -> 0.01
- link ring_sensor_4_link: mass 0 -> 0.01
- link thumb_sensor_2_link: mass 0 -> 0.01
- link thumb_sensor_3_link: mass 0 -> 0.01
